File: RasPi-BplusHAT.brd (EAGLE design)
At the start: 65 x 56 mm, 23 parts, among them K1 PIN20X2, K2 FSMR, K3 FSMR, K6 FSMR, U1 EEPROM24, U2 MCP3208-BI/SL, U3 TLC5615CD, U4 TLC5615CD, U5 ATMEGA32U4-AU, X1 1751251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

Commit message: Add files via upload
Parts:
- added IC1: LP2950CDT-3.3, v-reg:DPACK
- added JP1: (no value), pinhead:1_05X2MM
- added LED1, LED2, LED3: (no value), led:CHIPLED_1206
- added Q1: (no value), crystal:HC49UP
- moved OK3 15.1 mm to (51.4, 6.43)
- moved K6 9.40 mm to (22.6, 12.7)
- moved K2 9.40 mm to (30.9, 12.9)
- moved K3 9.27 mm to (39.2, 12.9)
- moved OK2 3.95 mm to (51.2, 18.9)
- moved U5 1.40 mm to (33.9, 35.3), flipped to the bottom
- moved OK1 1.30 mm to (60.4, 13.7)
- moved CFG 1.05 mm to (60.0, 34.2)
- moved X4 0.25 mm to (4.49, 13.1)
Routing:
- net N$3: track 0.00 -> 14.6 mm
- net +3V3: track 40.9 -> 51.8 mm, vias 0 -> 1
