File: RasPi-BplusHAT.sch (EAGLE design)
At the start: 21 parts, among them K1 PIN20X2, K2 FSMR, K3 FSMR, K6 FSMR, U1 EEPROM24, U2 MCP3208-BI/SL, U3 TLC5615CD, U4 TLC5615CD, U5 ATMEGA32U4-AU, X1 1751251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

Commit message: Add files via upload
Parts:
- added IC1: LP2950CDT-3.3, v-reg:LP2950CDT-3.3
- added JP1: (no value), pinhead:PINHD-1X55X2MM
- added LED1, LED2, LED3: (no value), led:LEDCHIPLED_1206
- added Q1: (no value), crystal:CRYSTALHC49UP
Changed lines of the file:
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@@
 <part name="U4" library="TLC5615CD" deviceset="TLC5615CD" device=""/>
 <part name="U5" library="ATMEGA32U4-AU" deviceset="ATMEGA32U4-AU" device=""/>
+<part name="IC1" library="v-reg" library_urn="urn:adsk.eagle:library:409" deviceset="LP2950?*" device="CDT" package3d_urn="urn:adsk.eagle:package:30369/1" technology="-3.3"/>
+<part name="JP1" library="pinhead" library_urn="urn:adsk.eagle:library:325" deviceset="PINHD-1X5" device="5X2MM" package3d_urn="urn:adsk.eagle:package:22466/2"/>
+<part name="LED1" library="led" library_urn="urn:adsk.eagle:library:259" deviceset="LED" device="CHIPLED_1206" package3d_urn="urn:adsk.eagle:package:15823/2"/>
+<part name="LED2" library="led" library_urn="urn:adsk.eagle:library:259" deviceset="LED" device="CHIPLED_1206" package3d_urn="urn:adsk.eagle:package:15823/2"/>
+<part name="LED3" library="led" library_urn="urn:adsk.eagle:library:259" deviceset="LED" device="CHIPLED_1206" package3d_urn="urn:adsk.eagle:package:15823/2"/>
+<part name="Q1" library="crystal" library_urn="urn:adsk.eagle:library:204" deviceset="CRYSTAL" device="HC49UP" package3d_urn="urn:adsk.eagle:package:12078/1"/>
 </parts>
 <sheets>
@@
 <instance part="U4" gate="A" x="160.02" y="50.8"/>
 <instance part="U5" gate="A" x="243.84" y="134.62"/>
+<instance part="IC1" gate="G$1" x="337.82" y="241.3"/>
+<instance part="JP1" gate="A" x="345.44" y="137.16"/>
+<instance part="LED1" gate="G$1" x="314.96" y="157.48"/>
+<instance part="LED2" gate="G$1" x="317.5" y="139.7"/>
+<instance part="LED3" gate="G$1" x="317.5" y="121.92"/>
+<instance part="Q1" gate="G$1" x="210.82" y="157.48"/>
 </instances>
 <busses>
